Commit message: added color to the bot

File: src/walle_description/urdf/materials.xacro (robot description, xacro)
@@ -4,3 +4,9 @@
   <color rgba="0.700 0.700 0.700 1.000"/>
 </material>
+<material name="black">
+  <color rgba="0.01 0.01 0.01 1"/>
+</material>
+<material name="yellow">
+  <color rgba="1.0 1.0 0.0 1"/>
+</material>
 </robot>

File: src/walle_description/urdf/walle.xacro (robot description, xacro)
@@ -16,5 +16,5 @@
       <mesh filename="file://$(find walle_description)/meshes/base_link.stl" scale="0.001 0.001 0.001"/>
     </geometry>
-    <material name="silver"/>
+    <material name="yellow"/>
   </visual>
   <collision>
@@ -36,5 +36,5 @@
       <mesh filename="file://$(find walle_description)/meshes/left_wheel_1.stl" scale="0.001 0.001 0.001"/>
     </geometry>
-    <material name="silver"/>
+    <material name="black"/>
   </visual>
   <collision>
@@ -56,5 +56,5 @@
       <mesh filename="file://$(find walle_description)/meshes/right_wheel_1.stl" scale="0.001 0.001 0.001"/>
     </geometry>
-    <material name="silver"/>
+    <material name="black"/>
   </visual>
   <collision>
@@ -96,5 +96,5 @@
       <mesh filename="file://$(find walle_description)/meshes/lidar_1.stl" scale="0.001 0.001 0.001"/>
     </geometry>
-    <material name="silver"/>
+    <material name="black"/>
   </visual>
   <collision>

File: src/walle_description/urdf/walle_gazebo.xacro (robot description, xacro)
@@ -1,45 +1,46 @@
 <?xml version="1.0" ?>
-<robot name="walle" xmlns:xacro="http://www.ros.org/wiki/xacro" >
-<xacro:property name="body_color" value="Gazebo/Silver" />
-<gazebo reference="left_wheel_1">
-  <material>${body_color}</material>
-  <mu1>1000000000000000.0</mu1>
-  <mu2>1000000000000000.0</mu2>
-  <kp>1000000000000.0</kp>
-  <kd>10.0</kd>
-  <minDepth>0.001</minDepth>
-  <maxVel>0.1</maxVel>
-  <fdir1>1 0 0</fdir1>
-</gazebo>
-<gazebo reference="right_wheel_1">
-  <material>${body_color}</material>
-  <mu1>1000000000000000.0</mu1>
-  <mu2>1000000000000000.0</mu2>
-  <kp>1000000000000.0</kp>
-  <kd>10.0</kd>
-  <minDepth>0.001</minDepth>
-  <maxVel>0.1</maxVel>
-  <fdir1>1 0 0</fdir1>
-</gazebo>
-<gazebo reference="caster_wheel_1">
-  <material>${body_color}</material>
-  <mu1>0.1</mu1>
-  <mu2>0.1</mu2>
-  <kp>1000000.0</kp>
-  <kd>100.0</kd>
-  <minDepth>0.001</minDepth>
-  <maxVel>0.1</maxVel>
-</gazebo>
-<gazebo>
-  <xacro:if value="$(arg is_ignition)">
-    <plugin filename="ign_ros2_control-system" name="ign_ros2_control::IgnitionROS2ControlPlugin">
-      <parameters>$(find walle_controller)/config/walle_controllers.yaml</parameters>
-    </plugin>
-  </xacro:if>
-  <xacro:unless value="$(arg is_ignition)">
-    <plugin filename="gz_ros2_control-system" name="gz_ros2_control::GazeboSimROS2ControlPlugin">
-      <parameters>$(find walle_controller)/config/walle_controllers.yaml</parameters>
-    </plugin>
-  </xacro:unless>
-</gazebo>
+<robot name="walle" xmlns:xacro="http://www.ros.org/wiki/xacro">
+  <xacro:property name="body_color" value="Gazebo/Yellow" />
+  <xacro:property name="wheel_color" value="Gazebo/Black" />
+  <gazebo reference="left_wheel_1">
+    <material>${wheel_color}</material>
+    <mu1>1000000000000000.0</mu1>
+    <mu2>1000000000000000.0</mu2>
+    <kp>1000000000000.0</kp>
+    <kd>10.0</kd>
+    <minDepth>0.001</minDepth>
+    <maxVel>0.1</maxVel>
+    <fdir1>1 0 0</fdir1>
+  </gazebo>
+  <gazebo reference="right_wheel_1">
+    <material>${wheel_color}</material>
+    <mu1>1000000000000000.0</mu1>
+    <mu2>1000000000000000.0</mu2>
+    <kp>1000000000000.0</kp>
+    <kd>10.0</kd>
+    <minDepth>0.001</minDepth>
+    <maxVel>0.1</maxVel>
+    <fdir1>1 0 0</fdir1>
+  </gazebo>
+  <gazebo reference="caster_wheel_1">
+    <material>${body_color}</material>
+    <mu1>0.1</mu1>
+    <mu2>0.1</mu2>
+    <kp>1000000.0</kp>
+    <kd>100.0</kd>
+    <minDepth>0.001</minDepth>
+    <maxVel>0.1</maxVel>
+  </gazebo>
+  <gazebo>
+    <xacro:if value="$(arg is_ignition)">
+      <plugin filename="ign_ros2_control-system" name="ign_ros2_control::IgnitionROS2ControlPlugin">
+        <parameters>$(find walle_controller)/config/walle_controllers.yaml</parameters>
+      </plugin>
+    </xacro:if>
+    <xacro:unless value="$(arg is_ignition)">
+      <plugin filename="gz_ros2_control-system" name="gz_ros2_control::GazeboSimROS2ControlPlugin">
+        <parameters>$(find walle_controller)/config/walle_controllers.yaml</parameters>
+      </plugin>
+    </xacro:unless>
+  </gazebo>
 </robot>
