Commit message: added imu

File: src/walle_description/urdf/walle.xacro (robot description, xacro)
@@ -105,4 +105,24 @@
   </collision>
 </link>
+<link name="imu_link">
+  <inertial>
+    <origin xyz="-8.696423535459186e-08 -3.511515006549004e-08 -0.0024998122926913197" rpy="0 0 0"/>
+    <mass value="0.007290803052000012"/>
+    <inertia ixx="0.0" iyy="0.0" izz="0.0" ixy="-0.0" iyz="0.0" ixz="0.0"/>
+  </inertial>
+  <visual>
+    <origin xyz="-0.089668 -0.161242 -0.089797" rpy="0 0 0"/>
+    <geometry>
+      <mesh filename="file://$(find walle_description)/meshes/imu_1.stl" scale="0.001 0.001 0.001"/>
+    </geometry>
+    <material name="silver"/>
+  </visual>
+  <collision>
+    <origin xyz="-0.089668 -0.161242 -0.089797" rpy="0 0 0"/>
+    <geometry>
+      <mesh filename="file://$(find walle_description)/meshes/imu_1.stl" scale="0.001 0.001 0.001"/>
+    </geometry>
+  </collision>
+</link>
 <joint name="left_wheel_joint" type="continuous">
   <origin xyz="0.055171 0.2712 0.054001" rpy="0 0 0"/>
@@ -127,3 +147,8 @@
   <child link="lidar_1"/>
 </joint>
+<joint name="imu_joint" type="fixed">
+  <origin xyz="0.089668 0.161242 0.089797" rpy="0 0 0"/>
+  <parent link="base_link"/>
+  <child link="imu_link"/>
+</joint>
 </robot>

File: src/walle_description/urdf/walle_gazebo.xacro (robot description, xacro)
@@ -50,5 +50,5 @@
     </xacro:unless>
   </gazebo>
-  <!-- <gazebo reference="imu_link">
+  <gazebo reference="imu_link">
     <sensor name="imu" type="imu">
       <always_on>true</always_on>
@@ -99,4 +99,4 @@
       </imu>
     </sensor>
-  </gazebo> -->
+  </gazebo>
 </robot>

Commit message: rviz

File: src/walle_description/urdf/walle.xacro (robot description, xacro)
@@ -6,4 +6,5 @@
 <xacro:include filename="$(find walle_description)/urdf/walle_ros2_control.xacro" />
 <xacro:include filename="$(find walle_description)/urdf/walle_gazebo.xacro" />
+ <link name="base_footprint"/>
 <link name="base_link">
   <inertial>
@@ -126,4 +127,9 @@
   </collision>
 </link>
+<joint name="base_joint" type="fixed">
+  <parent link="base_footprint"/>
+  <child link="base_link" />
+  <origin xyz="0 0 0" rpy="0 0 0"/>
+</joint>
 <joint name="left_wheel_joint" type="continuous">
   <origin xyz="0.055171 0.2712 0.054001" rpy="0 0 0"/>

Commit message: added 2D laser simulated

File: src/walle_description/urdf/walle.xacro (robot description, xacro)
@@ -6,5 +6,5 @@
 <xacro:include filename="$(find walle_description)/urdf/walle_ros2_control.xacro" />
 <xacro:include filename="$(find walle_description)/urdf/walle_gazebo.xacro" />
- <link name="base_footprint"/>
+<!-- <link name="base_footprint"/> -->
 <link name="base_link">
   <inertial>
@@ -87,5 +87,5 @@
   </collision>
 </link>
-<link name="lidar_1">
+<link name="laser_link">
   <inertial>
     <origin xyz="-8.696423536846964e-08 -2.808509075580279e-07 0.009718373123905832" rpy="0 0 0"/>
@@ -127,9 +127,9 @@
   </collision>
 </link>
-<joint name="base_joint" type="fixed">
+<!-- <joint name="base_joint" type="fixed">
   <parent link="base_footprint"/>
   <child link="base_link" />
   <origin xyz="0 0 0" rpy="0 0 0"/>
-</joint>
+</joint> -->
 <joint name="left_wheel_joint" type="continuous">
   <origin xyz="0.055171 0.2712 0.054001" rpy="0 0 0"/>
@@ -149,8 +149,8 @@
   <child link="caster_wheel_1"/>
 </joint>
-<joint name="lidar_joint" type="fixed">
+<joint name="laser_joint" type="fixed">
   <origin xyz="0.112168 0.16141 0.179797" rpy="0 0 0"/>
   <parent link="base_link"/>
-  <child link="lidar_1"/>
+  <child link="laser_link"/>
 </joint>
 <joint name="imu_joint" type="fixed">

File: src/walle_description/urdf/walle_gazebo.xacro (robot description, xacro)
@@ -40,4 +40,7 @@
       <plugin filename="ignition-gazebo-imu-system" name="ignition::gazebo::systems::Imu">
       </plugin>
+      <plugin filename="ignition-gazebo-sensors-system" name="ignition::gazebo::systems::Sensors">
+        <render_engine>ogre2</render_engine>
+      </plugin>
     </xacro:if>
 <!-- ROS2 iron or above-->
@@ -47,4 +50,7 @@
       </plugin>
       <plugin filename="gz-sim-imu-system" name="gz::sim::systems::Imu">
+      </plugin>
+      <plugin filename="gz-sim-sensors-system" name="gz::sim::systems::Sensors">
+        <render_engine>ogre2</render_engine>
       </plugin>
     </xacro:unless>
@@ -100,3 +106,33 @@
     </sensor>
   </gazebo>
+ <!-- 2D Laser Sensor -->
+  <gazebo reference="laser_link">
+    <sensor name="lidar" type="gpu_lidar">
+      <always_on>true</always_on>
+      <visualize>true</visualize>
+      <topic>scan</topic>
+      <update_rate>5</update_rate>
+      <gz_frame_id>laser_link</gz_frame_id>
+      <lidar>
+        <scan>
+          <horizontal>
+            <samples>360</samples>
+            <resolution>1.00000</resolution>
+            <min_angle>0.000000</min_angle>
+            <max_angle>6.280000</max_angle>
+          </horizontal>
+        </scan>
+        <range>
+          <min>0.120000</min>
+          <max>12.0</max>
+          <resolution>0.02</resolution>
+        </range>
+        <noise>
+          <type>gaussian</type>
+          <mean>0.0</mean>
+          <stddev>0.01</stddev>
+        </noise>
+      </lidar>
+    </sensor>
+  </gazebo>
 </robot>

Commit message: working simualted lidar

File: src/walle_description/urdf/walle.xacro (robot description, xacro)
@@ -6,8 +6,13 @@
 <xacro:include filename="$(find walle_description)/urdf/walle_ros2_control.xacro" />
 <xacro:include filename="$(find walle_description)/urdf/walle_gazebo.xacro" />
-<!-- <link name="base_footprint"/> -->
+<!-- <link name="base_footprint"/>
+<joint name="base_joint" type="fixed">
+  <parent link="base_footprint"/>
+  <child link="base_link" />
+  <origin xyz="0 0 0" rpy="0 0 0"/>
+</joint> -->
 <link name="base_link">
   <inertial>
-    <origin xyz="0.11032812925913082 0.16143345897542147 0.1194833264776962" rpy="0 0 0"/>
+    <origin xyz="-0.00045685530729292265 0.0004136281243083317 0.11948332647769622" rpy="0 0 0"/>
     <mass value="4.791704659790887"/>
     <inertia ixx="0.036131" iyy="0.02501" izz="0.044487" ixy="0.0" iyz="5e-06" ixz="-5.5e-05"/>
@@ -29,10 +34,10 @@
 <link name="left_wheel_1">
   <inertial>
-    <origin xyz="3.19240895607642e-07 0.025000458514719714 1.8088619061634725e-07" rpy="0 0 0"/>
+    <origin xyz="3.3467447201757095e-07 0.024999627663606278 1.808861906857362e-07" rpy="0 0 0"/>
     <mass value="3.5956470398131257"/>
     <inertia ixx="0.00337" iyy="0.005242" izz="0.00337" ixy="-0.0" iyz="0.0" ixz="0.0"/>
   </inertial>
   <visual>
-    <origin xyz="-0.055171 -0.2712 -0.054001" rpy="0 0 0"/>
+    <origin xyz="0.055614 -0.110181 -0.054001" rpy="0 0 0"/>
     <geometry>
       <mesh filename="file://$(find walle_description)/meshes/left_wheel_1.stl" scale="0.001 0.001 0.001"/>
@@ -41,5 +46,5 @@
   </visual>
   <collision>
-    <origin xyz="-0.055171 -0.2712 -0.054001" rpy="0 0 0"/>
+    <origin xyz="0.055614 -0.110181 -0.054001" rpy="0 0 0"/>
     <geometry>
       <mesh filename="file://$(find walle_description)/meshes/left_wheel_1.stl" scale="0.001 0.001 0.001"/>
@@ -49,10 +54,10 @@
 <link name="right_wheel_1">
   <inertial>
-    <origin xyz="3.1924089567009206e-07 -0.02500022053398937 1.8088619049144716e-07" rpy="0 0 0"/>
+    <origin xyz="3.346744719828765e-07 -0.025000051385102237 1.8088619053308053e-07" rpy="0 0 0"/>
     <mass value="3.5956470398131253"/>
-    <inertia ixx="0.00337" iyy="0.005242" izz="0.00337" ixy="0.0" iyz="0.0" ixz="0.0"/>
+    <inertia ixx="0.00337" iyy="0.005242" izz="0.00337" ixy="0.0" iyz="0.0" ixz="-0.0"/>
   </inertial>
   <visual>
-    <origin xyz="-0.055171 -0.051801 -0.054001" rpy="0 0 0"/>
+    <origin xyz="0.055614 0.109219 -0.054001" rpy="0 0 0"/>
     <geometry>
       <mesh filename="file://$(find walle_description)/meshes/right_wheel_1.stl" scale="0.001 0.001 0.001"/>
@@ -61,5 +66,5 @@
   </visual>
   <collision>
-    <origin xyz="-0.055171 -0.051801 -0.054001" rpy="0 0 0"/>
+    <origin xyz="0.055614 0.109219 -0.054001" rpy="0 0 0"/>
     <geometry>
       <mesh filename="file://$(find walle_description)/meshes/right_wheel_1.stl" scale="0.001 0.001 0.001"/>
@@ -69,10 +74,10 @@
 <link name="caster_wheel_1">
   <inertial>
-    <origin xyz="-8.696423534071407e-08 -2.8085090747476116e-07 -0.04496975521572785" rpy="0 0 0"/>
+    <origin xyz="-7.153065921527979e-08 -1.1170202059618186e-07 -0.04496975521572788" rpy="0 0 0"/>
     <mass value="0.4982856545913868"/>
-    <inertia ixx="0.000365" iyy="0.000365" izz="5.5e-05" ixy="-0.0" iyz="0.0" ixz="-0.0"/>
+    <inertia ixx="0.000365" iyy="0.000365" izz="5.5e-05" ixy="0.0" iyz="0.0" ixz="-0.0"/>
   </inertial>
   <visual>
-    <origin xyz="-0.212168 -0.16141 -0.094797" rpy="0 0 0"/>
+    <origin xyz="-0.101383 -0.00039 -0.094797" rpy="0 0 0"/>
     <geometry>
       <mesh filename="file://$(find walle_description)/meshes/caster_wheel_1.stl" scale="0.001 0.001 0.001"/>
@@ -81,5 +86,5 @@
   </visual>
   <collision>
-    <origin xyz="-0.212168 -0.16141 -0.094797" rpy="0 0 0"/>
+    <origin xyz="-0.101383 -0.00039 -0.094797" rpy="0 0 0"/>
     <geometry>
       <mesh filename="file://$(find walle_description)/meshes/caster_wheel_1.stl" scale="0.001 0.001 0.001"/>
@@ -89,10 +94,10 @@
 <link name="laser_link">
   <inertial>
-    <origin xyz="-8.696423536846964e-08 -2.808509075580279e-07 0.009718373123905832" rpy="0 0 0"/>
+    <origin xyz="-7.153065918145268e-08 -1.1170202091591308e-07 0.009718373123905694" rpy="0 0 0"/>
     <mass value="0.5843654094095093"/>
-    <inertia ixx="0.000193" iyy="0.000193" izz="0.000348" ixy="-0.0" iyz="0.0" ixz="-0.0"/>
+    <inertia ixx="0.000193" iyy="0.000193" izz="0.000348" ixy="0.0" iyz="0.0" ixz="-0.0"/>
   </inertial>
   <visual>
-    <origin xyz="-0.112168 -0.16141 -0.179797" rpy="0 0 0"/>
+    <origin xyz="-0.001383 -0.00039 -0.179797" rpy="0 0 0"/>
     <geometry>
       <mesh filename="file://$(find walle_description)/meshes/lidar_1.stl" scale="0.001 0.001 0.001"/>
@@ -101,5 +106,5 @@
   </visual>
   <collision>
-    <origin xyz="-0.112168 -0.16141 -0.179797" rpy="0 0 0"/>
+    <origin xyz="-0.001383 -0.00039 -0.179797" rpy="0 0 0"/>
     <geometry>
       <mesh filename="file://$(find walle_description)/meshes/lidar_1.stl" scale="0.001 0.001 0.001"/>
@@ -109,10 +114,10 @@
 <link name="imu_link">
   <inertial>
-    <origin xyz="-8.696423535459186e-08 -3.511515006549004e-08 -0.0024998122926913197" rpy="0 0 0"/>
+    <origin xyz="-7.153065904527689e-08 1.3403373669393544e-07 -0.0024998122926913197" rpy="0 0 0"/>
     <mass value="0.007290803052000012"/>
     <inertia ixx="0.0" iyy="0.0" izz="0.0" ixy="-0.0" iyz="0.0" ixz="0.0"/>
   </inertial>
   <visual>
-    <origin xyz="-0.089668 -0.161242 -0.089797" rpy="0 0 0"/>
+    <origin xyz="0.021117 -0.000222 -0.089797" rpy="0 0 0"/>
     <geometry>
       <mesh filename="file://$(find walle_description)/meshes/imu_1.stl" scale="0.001 0.001 0.001"/>
@@ -121,5 +126,5 @@
   </visual>
   <collision>
-    <origin xyz="-0.089668 -0.161242 -0.089797" rpy="0 0 0"/>
+    <origin xyz="0.021117 -0.000222 -0.089797" rpy="0 0 0"/>
     <geometry>
       <mesh filename="file://$(find walle_description)/meshes/imu_1.stl" scale="0.001 0.001 0.001"/>
@@ -127,33 +132,28 @@
   </collision>
 </link>
-<!-- <joint name="base_joint" type="fixed">
-  <parent link="base_footprint"/>
-  <child link="base_link" />
-  <origin xyz="0 0 0" rpy="0 0 0"/>
-</joint> -->
 <joint name="left_wheel_joint" type="continuous">
-  <origin xyz="0.055171 0.2712 0.054001" rpy="0 0 0"/>
+  <origin xyz="-0.055614 0.110181 0.054001" rpy="0 0 0"/>
   <parent link="base_link"/>
   <child link="left_wheel_1"/>
-  <axis xyz="0.0 1.0 0.0"/>
+  <axis xyz="-0.0 1.0 0.0"/>
 </joint>
 <joint name="right_wheel_joint" type="continuous">
-  <origin xyz="0.055171 0.051801 0.054001" rpy="0 0 0"/>
+  <origin xyz="-0.055614 -0.109219 0.054001" rpy="0 0 0"/>
   <parent link="base_link"/>
   <child link="right_wheel_1"/>
-  <axis xyz="0.0 1.0 0.0"/>
+  <axis xyz="0.0 -1.0 -0.0"/>
 </joint>
 <joint name="caster_wheel_joint" type="fixed">
-  <origin xyz="0.212168 0.16141 0.094797" rpy="0 0 0"/>
+  <origin xyz="0.101383 0.00039 0.094797" rpy="0 0 0"/>
   <parent link="base_link"/>
   <child link="caster_wheel_1"/>
 </joint>
 <joint name="laser_joint" type="fixed">
-  <origin xyz="0.112168 0.16141 0.179797" rpy="0 0 0"/>
+  <origin xyz="0.001383 0.00039 0.179797" rpy="0 0 0"/>
   <parent link="base_link"/>
   <child link="laser_link"/>
 </joint>
 <joint name="imu_joint" type="fixed">
-  <origin xyz="0.089668 0.161242 0.089797" rpy="0 0 0"/>
+  <origin xyz="-0.021117 0.000222 0.089797" rpy="0 0 0"/>
   <parent link="base_link"/>
   <child link="imu_link"/>

File: src/walle_description/urdf/walle_gazebo.xacro (robot description, xacro)
@@ -124,5 +124,5 @@
         </scan>
         <range>
-          <min>0.120000</min>
+          <min>0.40</min>
           <max>12.0</max>
           <resolution>0.02</resolution>

Commit message: .

File: src/walle_description/urdf/walle.xacro (robot description, xacro)
@@ -136,5 +136,5 @@
   <parent link="base_link"/>
   <child link="left_wheel_1"/>
-  <axis xyz="-0.0 1.0 0.0"/>
+  <axis xyz="0.0 1.0 0.0"/>
 </joint>
 <joint name="right_wheel_joint" type="continuous">
@@ -142,5 +142,5 @@
   <parent link="base_link"/>
   <child link="right_wheel_1"/>
-  <axis xyz="0.0 -1.0 -0.0"/>
+  <axis xyz="0.0 1.0 0.0"/>
 </joint>
 <joint name="caster_wheel_joint" type="fixed">

File: src/walle_description/urdf/walle_gazebo.xacro (robot description, xacro)
@@ -124,5 +124,5 @@
         </scan>
         <range>
-          <min>0.40</min>
+          <min>0.20</min>
           <max>12.0</max>
           <resolution>0.02</resolution>

Commit message: updated urdf

File: src/walle_description/urdf/walle.xacro (robot description, xacro)
@@ -6,10 +6,5 @@
 <xacro:include filename="$(find walle_description)/urdf/walle_ros2_control.xacro" />
 <xacro:include filename="$(find walle_description)/urdf/walle_gazebo.xacro" />
-<!-- <link name="base_footprint"/>
-<joint name="base_joint" type="fixed">
-  <parent link="base_footprint"/>
-  <child link="base_link" />
-  <origin xyz="0 0 0" rpy="0 0 0"/>
-</joint> -->
+<link name="base_footprint"/>
 <link name="base_link">
   <inertial>
@@ -19,5 +14,5 @@
   </inertial>
   <visual>
-    <origin xyz="0 0 0" rpy="0 0 0"/>
+    <origin xyz="0 0 -0.054001" rpy="0 0 0"/>
     <geometry>
       <mesh filename="file://$(find walle_description)/meshes/base_link.stl" scale="0.001 0.001 0.001"/>
@@ -32,4 +27,9 @@
   </collision>
 </link>
+<joint name="base_joint" type="fixed">
+  <parent link="base_footprint"/>
+  <child link="base_link" />
+  <origin xyz="0 0 0.054001" rpy="0 0 0"/>
+</joint>
 <link name="left_wheel_1">
   <inertial>
@@ -133,5 +133,5 @@
 </link>
 <joint name="left_wheel_joint" type="continuous">
-  <origin xyz="-0.055614 0.110181 0.054001" rpy="0 0 0"/>
+  <origin xyz="-0.055614 0.110181 0" rpy="0 0 0"/>
   <parent link="base_link"/>
   <child link="left_wheel_1"/>
@@ -139,5 +139,5 @@
 </joint>
 <joint name="right_wheel_joint" type="continuous">
-  <origin xyz="-0.055614 -0.109219 0.054001" rpy="0 0 0"/>
+  <origin xyz="-0.055614 -0.109219 0" rpy="0 0 0"/>
   <parent link="base_link"/>
   <child link="right_wheel_1"/>
@@ -145,15 +145,15 @@
 </joint>
 <joint name="caster_wheel_joint" type="fixed">
-  <origin xyz="0.101383 0.00039 0.094797" rpy="0 0 0"/>
+  <origin xyz="0.101383 0.00039 0.0400" rpy="0 0 0"/>
   <parent link="base_link"/>
   <child link="caster_wheel_1"/>
 </joint>
-<joint name="laser_joint" type="fixed">
-  <origin xyz="0.001383 0.00039 0.179797" rpy="0 0 0"/>
+<joint name="lidar_joint" type="fixed">
+  <origin xyz="0.001383 0.00039 0.12600" rpy="0 0 0"/>
   <parent link="base_link"/>
   <child link="laser_link"/>
 </joint>
 <joint name="imu_joint" type="fixed">
-  <origin xyz="-0.021117 0.000222 0.089797" rpy="0 0 0"/>
+  <origin xyz="-0.021117 0.000222 0.0600" rpy="0 0 0"/>
   <parent link="base_link"/>
   <child link="imu_link"/>
